File: slidepot/hardware/slidepot-45/slidepot-45.kicad_sch (KiCad schematic)
At the start: 3 parts, among them J1 Conn_01x05_Male, J2 Conn_01x02

Commit message: Update slideot-45 footprint
Parts:
- RV1: footprint Potentiometer_THT:Potentiometer_Bourns_PTA6043_Single_Slide -> Potentiometer_THT:Potentiometer_Bourns_PTA4543_Single_Slide
Changed lines of the file:
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@@
       (effects (font (size 1.27 1.27)) (justify right))
     )
-    (property "Footprint" "Potentiometer_THT:Potentiometer_Bourns_PTA6043_Single_Slide" (id 2) (at 128.27 76.2 0)
+    (property "Footprint" "Potentiometer_THT:Potentiometer_Bourns_PTA4543_Single_Slide" (id 2) (at 128.27 76.2 0)
       (effects (font (size 1.27 1.27)) hide)
     )
@@
     )
     (path "/9531b8f7-c21e-4d2d-a08b-fcb6e8903a99"
-      (reference "RV1") (unit 1) (value "R_Potentiometer") (footprint "Potentiometer_THT:Potentiometer_Bourns_PTA6043_Single_Slide")
+      (reference "RV1") (unit 1) (value "R_Potentiometer") (footprint "Potentiometer_THT:Potentiometer_Bourns_PTA4543_Single_Slide")
     )
   )
