File: slidepot/hardware/slidepot-60/slidepot-60.kicad_pcb (KiCad board)
At the start: 2 copper layers, 17.8 x 92.7 mm, 3 parts, among them J1 Conn_01x05_Male, J2 Conn_01x02

Commit message: Assign part numbers
Parts:
- added G***: LOGO, LOGO, B.Cu at (165.1, 82.5)
Other:
- board text added: "D.R.U.M. Slidepot 60mm Riser HW Design REV: 1.0 Layout REV: A Order No. P/N DRUM-SR-1060"

Commit message: Generate slidepot gerbers
Routing:
- net GND: track 2.47 -> 0.00 mm
Other:
- rule pad_to_mask_clearance: 0.05 -> 0
Changed lines of the file:
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@@
       (dielectric_constraints no)
     )
-    (pad_to_mask_clearance 0.05)
-    (solder_mask_min_width 0.2)
+    (pad_to_mask_clearance 0)
     (pcbplotparams
       (layerselection 0x00010fc_ffffffff)
@@
       (outputformat 1)
       (mirror false)
-      (drillshape 1)
+      (drillshape 0)
       (scaleselection 1)
-      (outputdirectory "")
+      (outputdirectory "gerb")
     )
   )
@@
   (segment (start 165.095 122.855) (end 166.85 124.61) (width 1.016) (layer "F.Cu") (net 3))
   (segment (start 165.095 45.72) (end 165.095 122.855) (width 1.016) (layer "F.Cu") (net 3))
-  (segment (start 165.1 122.86) (end 163.35 124.61) (width 1.016) (layer "B.Cu") (net 4))
   (zone (net 4) (net_name "GND") (layers F&B.Cu) (hatch edge 0.508)
     (connect_pads (clearance 0.508))
